File: eagle/GVSwire1.brd (EAGLE design)
At the start: 100 x 80 mm, 16 parts

Commit message: updated original paolo circuit
Parts:
- removed CONTROL: AYZ0202, SparkFun:AYZ0202
- removed LEFT, RIGHT: M01PTH_2MM, SparkFun:1X01_2MM
- removed ONOFF: (no value), SparkFun:SWITCH-SPDT
- added LEFT_IN, LEFT_OUT, RIGHT_IN, RIGHT_OUT: M01PTH_2MM, SparkFun:1X01_2MM
- 9VBATTERY: value (none) -> 9V
- moved R1 29.0 mm to (63.5, 7.62), turned to 180 degrees
- moved R2 26.2 mm to (63.5, 27.9), turned to 0 degrees
- moved R5 17.0 mm to (44.5, 7.62)
- moved Q4 14.8 mm to (50.8, 19.1)
- moved R4 14.0 mm to (27.9, 26.7)
- moved Q1 13.0 mm to (39.4, 36.8)
- moved R6 12.8 mm to (27.9, 31.8), turned to 180 degrees
- moved Q2 11.7 mm to (35.6, 19.1)
- moved Q3 10.9 mm to (48.3, 30.5)
- moved 9VBATTERY 5.24 mm to (3.81, 3.81), turned to 90 degrees
- moved REGULATOR 4.02 mm to (7.62, 44.5), turned to 270 degrees
- moved R3 3.59 mm to (27.9, 17.8)
Connections:
- removed net N$9: ONOFF.1, REGULATOR.P$1
- net GND: no longer CONTROL.1, CONTROL.6
- net LEFT: now also LEFT_IN.1; no longer CONTROL.5
- net N$11: now also RIGHT_OUT.1; no longer RIGHT.1
- net N$7: now also LEFT_OUT.1; no longer LEFT.1
- net RIGHT: now also RIGHT_IN.1; no longer CONTROL.2
- net VCC: now also REGULATOR.P$1; no longer CONTROL.3, CONTROL.4, ONOFF.2
Routing:
- net GND: track 63.1 -> 0.00 mm
- net LEFT: track 39.0 -> 0.00 mm, vias 1 -> 0
- net VCC: track 36.0 -> 0.00 mm
- net POT: track 25.4 -> 0.00 mm
- net N$5: track 23.1 -> 0.00 mm
- net N$2: track 18.8 -> 0.00 mm
- net N$9: track 17.9 -> 0.00 mm
- net N$3: track 17.7 -> 0.00 mm
- net RIGHT: track 16.7 -> 0.00 mm
- net N$6: track 14.6 -> 0.00 mm
- net N$4: track 11.3 -> 0.00 mm
- net N$1: track 7.37 -> 0.00 mm
- net N$7: track 4.66 -> 0.00 mm
- net N$11: track 4.60 -> 0.00 mm
Other:
- board text added: "+"
- board text added: "-"
- board text added: "10k or 100k potentiometer"
- board text added: "9V"
- board text added: "NPN"
