File: eagle/GVSwire1.sch (EAGLE design)
At the start: 16 parts

Commit message: updated original paolo circuit
Parts:
- removed CONTROL: AYZ0202, SparkFun:AYZ0202
- removed LEFT, RIGHT: M01PTH_2MM, SparkFun:M01PTH_2MM
- removed ONOFF: (no value), SparkFun:SWITCH-SPSTPTH
- added LEFT_IN, LEFT_OUT, RIGHT_IN, RIGHT_OUT: M01PTH_2MM, SparkFun:M01PTH_2MM
- 9VBATTERY: value (none) -> 9V
Connections:
- removed net N$9: ONOFF.O, REGULATOR.E
- net GND: no longer CONTROL.3, CONTROL.4
- net LEFT: now also LEFT_IN.1; no longer CONTROL.5
- net N$11: now also RIGHT_OUT.1; no longer RIGHT.1
- net N$7: now also LEFT_OUT.1; no longer LEFT.1
- net RIGHT: now also RIGHT_IN.1; no longer CONTROL.2
- net VCC: now also REGULATOR.E; no longer CONTROL.1, CONTROL.6, ONOFF.P
Changed lines of the file:
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@@
 <part name="R6" library="adafruit" deviceset="R-US_" device="FLIPFLOP7" value="1k"/>
 <part name="REGULATOR" library="SparkFun" deviceset="POT" device="" value="100k"/>
-<part name="CONTROL" library="SparkFun" deviceset="AYZ0202" device=""/>
-<part name="GND3" library="SparkFun" deviceset="GND" device=""/>
-<part name="P+2" library="SparkFun" deviceset="VCC" device=""/>
-<part name="P+3" library="SparkFun" deviceset="VCC" device=""/>
-<part name="LEFT" library="SparkFun" deviceset="M01" device="PTH_2MM"/>
-<part name="RIGHT" library="SparkFun" deviceset="M01" device="PTH_2MM"/>
-<part name="ONOFF" library="SparkFun" deviceset="SWITCH-SPST" device="PTH"/>
-<part name="9VBATTERY" library="SparkFun" deviceset="M02" device=""/>
+<part name="LEFT_OUT" library="SparkFun" deviceset="M01" device="PTH_2MM"/>
+<part name="RIGHT_OUT" library="SparkFun" deviceset="M01" device="PTH_2MM"/>
+<part name="9VBATTERY" library="SparkFun" deviceset="M02" device="" value="9V"/>
 <part name="GND2" library="SparkFun" deviceset="GND" device=""/>
 <part name="P+4" library="SparkFun" deviceset="VCC" device=""/>
+<part name="RIGHT_IN" library="SparkFun" deviceset="M01" device="PTH_2MM"/>
+<part name="LEFT_IN" library="SparkFun" deviceset="M01" device="PTH_2MM"/>
 </parts>
 <sheets>
@@
 <instance part="R6" gate="G$1" x="10.16" y="68.58" rot="R180"/>
 <instance part="REGULATOR" gate="G$1" x="35.56" y="83.82"/>
-<instance part="CONTROL" gate="G$1" x="-30.48" y="55.88" rot="R180"/>
-<instance part="GND3" gate="1" x="-43.18" y="58.42" rot="R270"/>
-<instance part="P+2" gate="1" x="-40.64" y="50.8"/>
-<instance part="P+3" gate="1" x="-40.64" y="63.5"/>
-<instance part="LEFT" gate="G$1" x="30.48" y="50.8" rot="R90"/>
-<instance part="RIGHT" gate="G$1" x="40.64" y="50.8" rot="R90"/>
-<instance part="ONOFF" gate="1" x="33.02" y="99.06" rot="R180"/>
+<instance part="LEFT_OUT" gate="G$1" x="30.48" y="45.72" rot="R90"/>
+<instance part="RIGHT_OUT" gate="G$1" x="40.64" y="45.72" rot="R90"/>
 <instance part="9VBATTERY" gate="G$1" x="0" y="91.44"/>
 <instance part="GND2" gate="1" x="10.16" y="86.36"/>
 <instance part="P+4" gate="1" x="10.16" y="96.52"/>
+<instance part="RIGHT_IN" gate="G$1" x="99.06" y="55.88" rot="R180"/>
+<instance part="LEFT_IN" gate="G$1" x="-22.86" y="55.88"/>
 </instances>
 <busses>
@@
 <net name="VCC" class="0">
 <segment>
-<wire x1="-35.56" y1="50.8" x2="-40.64" y2="50.8" width="0.2032" layer="91"/>
-<pinref part="CONTROL" gate="G$1" pin="1"/>
-<pinref part="P+2" gate="1" pin="VCC"/>
-</segment>
-<segment>
-<wire x1="-35.56" y1="63.5" x2="-40.64" y2="63.5" width="0.2032" layer="91"/>
-<pinref part="CONTROL" gate="G$1" pin="6"/>
-<pinref part="P+3" gate="1" pin="VCC"/>
-</segment>
-<segment>
 <wire x1="35.56" y1="99.06" x2="35.56" y2="104.14" width="0.2032" layer="91"/>
-<junction x="35.56" y="99.06"/>
-<pinref part="ONOFF" gate="1" pin="P"/>
 <pinref part="P+1" gate="1" pin="VCC"/>
+<pinref part="REGULATOR" gate="G$1" pin="E"/>
+<wire x1="35.56" y1="99.06" x2="35.56" y2="91.44" width="0.1524" layer="91"/>
 </segment>
 <segment>
@@
 <net name="LEFT" class="0">
 <segment>
-<wire x1="-25.4" y1="60.96" x2="-17.78" y2="60.96" width="0.2032" layer="91"/>
-<label x="-17.78" y="60.96" size="1.778" layer="95"/>
-<pinref part="CONTROL" gate="G$1" pin="5"/>
-</segment>
-<segment>
 <wire x1="-2.54" y1="68.58" x2="5.08" y2="68.58" width="0.2032" layer="91"/>
 <wire x1="-2.54" y1="68.58" x2="-2.54" y2="55.88" width="0.2032" layer="91"/>
@@
 <wire x1="-2.54" y1="38.1" x2="66.04" y2="38.1" width="0.2032" layer="91"/>
 <wire x1="66.04" y1="48.26" x2="66.04" y2="38.1" width="0.2032" layer="91"/>
-<wire x1="-2.54" y1="55.88" x2="5.08" y2="55.88" width="0.2032" layer="91"/>
-<junction x="-2.54" y="55.88"/>
-<label x="7.62" y="55.88" size="1.778" layer="95"/>
 <pinref part="R6" gate="G$1" pin="2"/>
 <pinref part="R4" gate="G$1" pin="1"/>
+<pinref part="LEFT_IN" gate="G$1" pin="1"/>
+<wire x1="-15.24" y1="55.88" x2="-2.54" y2="55.88" width="0.1524" layer="91"/>
+<label x="-10.16" y="55.88" size="1.778" layer="95"/>
+<junction x="-2.54" y="55.88"/>
 </segment>
 </net>
@@
 <segment>
 <pinref part="R1" gate="G$1" pin="1"/>
-<pinref part="LEFT" gate="G$1" pin="1"/>
+<pinref part="LEFT_OUT" gate="G$1" pin="1"/>
+<wire x1="30.48" y1="53.34" x2="30.48" y2="58.42" width="0.1524" layer="91"/>
 </segment>
 </net>
@@
 <segment>
 <pinref part="R2" gate="G$1" pin="2"/>
-<pinref part="RIGHT" gate="G$1" pin="1"/>
+<pinref part="RIGHT_OUT" gate="G$1" pin="1"/>
+<wire x1="40.64" y1="53.34" x2="40.64" y2="58.42" width="0.1524" layer="91"/>
 </segment>
 </net>
@@
 <wire x1="76.2" y1="35.56" x2="76.2" y2="55.88" width="0.2032" layer="91"/>
 <wire x1="76.2" y1="55.88" x2="76.2" y2="68.58" width="0.2032" layer="91"/>
-<wire x1="76.2" y1="55.88" x2="81.28" y2="55.88" width="0.2032" layer="91"/>
+<wire x1="76.2" y1="55.88" x2="91.44" y2="55.88" width="0.2032" layer="91"/>
 <junction x="76.2" y="55.88"/>
-<label x="83.82" y="55.88" size="1.778" layer="95"/>
+<label x="76.2" y="55.88" size="1.778" layer="95"/>
 <pinref part="R3" gate="G$1" pin="2"/>
 <pinref part="R5" gate="G$1" pin="1"/>
-</segment>
-<segment>
-<wire x1="-25.4" y1="53.34" x2="-17.78" y2="53.34" width="0.2032" layer="91"/>
-<label x="-17.78" y="53.34" size="1.778" layer="95"/>
-<pinref part="CONTROL" gate="G$1" pin="2"/>
+<pinref part="RIGHT_IN" gate="G$1" pin="1"/>
 </segment>
 </net>
 <net name="GND" class="0">
-<segment>
-<wire x1="-35.56" y1="58.42" x2="-38.1" y2="58.42" width="0.2032" layer="91"/>
-<wire x1="-38.1" y1="58.42" x2="-40.64" y2="58.42" width="0.2032" layer="91"/>
-<wire x1="-35.56" y1="55.88" x2="-38.1" y2="55.88" width="0.2032" layer="91"/>
-<wire x1="-38.1" y1="55.88" x2="-38.1" y2="58.42" width="0.2032" layer="91"/>
-<pinref part="CONTROL" gate="G$1" pin="4"/>
-<pinref part="GND3" gate="1" pin="GND"/>
-<pinref part="CONTROL" gate="G$1" pin="3"/>
-</segment>
 <segment>
 <wire x1="20.32" y1="43.18" x2="20.32" y2="40.64" width="0.2032" layer="91"/>
@@
 </segment>
 </net>
-<net name="N$9" class="0">
-<segment>
-<wire x1="35.56" y1="93.98" x2="35.56" y2="91.44" width="0.1524" layer="91"/>
-<wire x1="27.94" y1="96.52" x2="27.94" y2="93.98" width="0.2032" layer="91"/>
-<wire x1="27.94" y1="93.98" x2="35.56" y2="93.98" width="0.2032" layer="91"/>
-<junction x="35.56" y="93.98"/>
-<pinref part="REGULATOR" gate="G$1" pin="E"/>
-<pinref part="ONOFF" gate="1" pin="O"/>
-</segment>
-</net>
